File: raicycle.kicad_sch (KiCad schematic)
At the start: 12 parts, among them J1 LiPo_Battery, J2 USB_B_Micro, U1 ESP32-S3-WROOM-1, U2 BME688, U3 VL53L0X

Commit message: Complete KiCad 8.0 schematic with all professor's suggestions implemented
Co-authored-by: 968096 <203631091+968096@users.noreply.github.com>
Parts:
- added C5: 100nF, Capacitor_SMD:C_0603_1608Metric, symbol Device:C
- added R3, R4: 10k, Resistor_SMD:R_0603_1608Metric, symbol Device:R
- added U4: BME688, Package_LGA:Bosch_LGA-8_3x3mm_P0.8mm_ClockwisePinNumbering, symbol Sensor_Environmental:BME688
- added U5: Grove_Wio-E5, Module:Grove_1x04_P2.54mm_Vertical, symbol Module:Grove_Wio-E5
- added U6: GPS_Air530, Module:Grove_1x04_P2.54mm_Vertical, symbol Module:GPS_Air530
Connections:
- net GND is gone; now on net +3V3: C1.2, C2.2, C3.2, C4.2, J1.2 (Pin_2), J2.5 (GND), U1.1 (GND), U2.1 (GND), U2.8 (GND), U3.1 (AVSSVCSEL), U3.9 (DNC)
- net +3V3: now also C5.2, R3.2, R4.2, U4.1 (GND), U4.8 (GND)
- new net: C5.1, U4.6 (VDDIO)
Other:
- note added: "Professor's Design Improvements Implemented: 1. I²C Pull-ups: 4.7k resistors on SDA/SCL lines 2. AVDD Analog Power Filtering: L1 (10uH) + C4 (10uF) 3. Power Decoupling: 100nF capacitors near each chip 4. Separate Power Rails: USB 5V vs 3.3V regulated 5. LiPo Battery Connection: J1 with proper handling 6. Pull-downs: 10k resistors on unused inputs 7. Clear Labeling: All signals properly labeled 8.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"
